File: frkbmb28.kicad_pcb (KiCad board)
At the start: 2 copper layers, 175 parts, among them P1 SHITTY_ADD_ON, P2 MCU_CONNECTOR, P3 SCL_JMP, P4 SDA_JMP, U1 IS31FL3741, U2 LIS2HH12

Commit message: more routing on prototype
Parts:
- moved R16 224.4 mm to (30.5, 36.8), turned to 180 degrees
- moved R27 211.3 mm to (30.5, 44.3), turned to 180 degrees
- moved R44 209.5 mm to (30.5, 57.1), turned to 180 degrees
- moved R35 208.3 mm to (30.5, 49.5), turned to 180 degrees
- moved R47 208.3 mm to (30.5, 59.7), turned to 180 degrees
- moved R30 208.2 mm to (30.5, 47.0), turned to 180 degrees
- moved R38 208.1 mm to (30.5, 52.1), turned to 180 degrees
- moved R10 208.0 mm to (30.5, 31.8), turned to 180 degrees
- moved R41 202.2 mm to (30.5, 54.6), turned to 180 degrees
- moved R19 202.1 mm to (30.5, 39.4), turned to 180 degrees
- moved R13 201.5 mm to (30.5, 34.3), turned to 180 degrees
- moved R22 201.4 mm to (30.5, 41.9), turned to 180 degrees
- moved R5 201.2 mm to (30.5, 29.2), turned to 180 degrees
- moved R26 179.2 mm to (72.8, 42.2)
- moved R11 174.8 mm to (77.8, 31.4)
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Connections:
- R40 pad 2: Net-(R40-Pad2) -> /CS31
- R41 pad 2: Net-(R41-Pad2) -> /CS32
- R42 pad 2: Net-(R42-Pad2) -> /CS33
Routing:
- net /CS37: track 0.00 -> 30.6 mm
- net /CS39: track 0.00 -> 27.5 mm
- net /CS34: track 0.00 -> 25.8 mm
- net /CS31: track 0.00 -> 23.9 mm
- net /CS36: track 0.00 -> 23.8 mm
- net /CS1: track 0.00 -> 21.6 mm
- net /CS28: track 0.00 -> 21.2 mm
- net /CS33: track 0.00 -> 19.9 mm
- net /CS25: track 0.00 -> 19.8 mm
- net /CS4: track 0.00 -> 18.5 mm
- net /CS22: track 0.00 -> 17.9 mm
- net /CS30: track 0.00 -> 17.6 mm
- net /CS10: track 0.00 -> 17.1 mm
- net /CS7: track 0.00 -> 16.8 mm
- net /CS13: track 0.00 -> 16.3 mm
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Other:
- board outline added: 99.1 x 99.1 mm
- net class Default: clearance 0.2 -> 0.127
- rule trace_clearance: 0.2 -> 0.127
