File: frkbmb28.sch (KiCad schematic (older format))
At the start: 133 parts

Commit message: work on prototype LED matrix
Parts:
- removed 10uF: C, symbol C
- removed JP? (x2): Jumper_NO_Small, symbol Jumper_NO_Small
- removed P?: CONN_01X12, symbol CONN_01X12
- added C1: 10uF, SMD_Packages:SMD-1210_Pol, symbol CP
- added P1: SHITTY_ADD_ON, Pin_Headers:Pin_Header_Straight_2x03, symbol CONN_02X03
- added P2: MCU_CONNECTOR, Pin_Headers:Pin_Header_Straight_1x18, symbol CONN_01X18
- added P3: SCL_JMP, Pin_Headers:Pin_Header_Straight_1x03, symbol CONN_01X03
- added P4: SDA_JMP, Pin_Headers:Pin_Header_Straight_1x03, symbol CONN_01X03
- added R1, R10, R11, R12, R13, R14, R15, R16, R17, R18, R19, R20, R21, R22, R23, R26, R27, R28, R29, R30, R31, R34, R35, R36, R37, R38, R39, R40, R41, R42, R43, R44, R45, R46, R47, R48, R5, R6, R8: R, Resistors_SMD:R_0805_HandSoldering, symbol R
- added R24, R25: 1k, Resistors_SMD:R_0603_HandSoldering, symbol R
- C2: renamed from 1uF; value C -> 1uF; footprint (none) -> Capacitors_SMD:C_0805_HandSoldering
- C3, C4: renamed from 100nF; value C -> 100nF; footprint (none) -> Capacitors_SMD:C_0603_HandSoldering
- D1, D10, D100, D101, D102, D103, D104, D105, D106, D107, D108, D109, D11, D110, D111, D112, D113, D114, D115, D116, D117, D12, D13, D14, D15, D16, D17, D18, D19, D2, D20, D21, D22, D23, D24, D25, D26, D27, D28, D29, D3, D30, D31, D32, D33, D34, D35, D36, D37, D38, D39, D4, D40, D41, D42, D43, D44, D45, D46, D47, D48, D49, D5, D50, D51, D52, D53, D54, D55, D56, D57, D58, D59, D6, D60, D61, D62, D63, D64, D65, D66, D67, D68, D69, D7, D70, D71, D72, D73, D74, D75, D76, D77, D78, D79, D8, D80, D81, D82, D83, D84, D85, D86, D87, D88, D89, D9, D90, D91, D92, D93, D94, D95, D96, D97, D98, D99: renamed from D?; footprint (none) -> frkbmb:0606_RGB_COMM_ANODE
- R2, R3, R32, R33: renamed from 1K; value R -> 1k; footprint (none) -> Resistors_SMD:R_0603_HandSoldering
- R4, R7: renamed from 100K; value R -> 100k; footprint (none) -> Resistors_SMD:R_0603_HandSoldering
- R9: renamed from 20K; value R -> 20k; footprint (none) -> Resistors_SMD:R_0603_HandSoldering
- U1: renamed from U?; footprint (none) -> frkbmb:IS31FL3741
- U2: renamed from U?; footprint (none) -> frkbmb:LIS2HH12
Connections:
- net +3V3: now also C1.1, P1.1 (P1), P2.1 (P1), R24.1, R25.1
- net CS: now also P2.12 (P12)
- net CS1: now also R1.2; no longer D2.2 (RK), D3.2 (RK), D4.2 (RK), D5.2 (RK), D6.2 (RK), D7.2 (RK), D8.2 (RK), D9.2 (RK)
- net CS10: now also R15.2; no longer D28.2 (RK), D29.2 (RK), D30.2 (RK), D31.2 (RK), D32.2 (RK), D33.2 (RK), D34.2 (RK), D35.2 (RK), D36.2 (RK)
- net CS11: now also R16.2; no longer D28.3 (GK), D29.3 (GK), D30.3 (GK), D31.3 (GK), D32.3 (GK), D33.3 (GK), D34.3 (GK), D35.3 (GK), D36.3 (GK)
- net CS12: now also R17.2; no longer D28.4 (BK), D29.4 (BK), D30.4 (BK), D31.4 (BK), D32.4 (BK), D33.4 (BK), D34.4 (BK), D35.4 (BK), D36.4 (BK)
- net CS13: now also R18.2; no longer D37.2 (RK), D38.2 (RK), D39.2 (RK), D40.2 (RK), D41.2 (RK), D42.2 (RK), D43.2 (RK), D44.2 (RK), D45.2 (RK)
- net CS14: now also R19.2; no longer D37.3 (GK), D38.3 (GK), D39.3 (GK), D40.3 (GK), D41.3 (GK), D42.3 (GK), D43.3 (GK), D44.3 (GK), D45.3 (GK)
- net CS15: now also R20.2; no longer D37.4 (BK), D38.4 (BK), D39.4 (BK), D40.4 (BK), D41.4 (BK), D42.4 (BK), D43.4 (BK), D44.4 (BK), D45.4 (BK)
- net CS16: now also R21.2; no longer D46.2 (RK), D47.2 (RK), D48.2 (RK), D49.2 (RK), D50.2 (RK), D51.2 (RK), D52.2 (RK), D53.2 (RK), D54.2 (RK)
- net CS17: now also R22.2; no longer D46.3 (GK), D47.3 (GK), D48.3 (GK), D49.3 (GK), D50.3 (GK), D51.3 (GK), D52.3 (GK), D53.3 (GK), D54.3 (GK)
- net CS18: now also R23.2; no longer D46.4 (BK), D47.4 (BK), D48.4 (BK), D49.4 (BK), D50.4 (BK), D51.4 (BK), D52.4 (BK), D53.4 (BK), D54.4 (BK)
- net CS19: now also R26.2; no longer D55.2 (RK), D56.2 (RK), D57.2 (RK), D58.2 (RK), D59.2 (RK), D60.2 (RK), D61.2 (RK), D62.2 (RK), D63.2 (RK)
- net CS2: now also R5.2; no longer D1.3 (GK), D2.3 (GK), D3.3 (GK), D4.3 (GK), D5.3 (GK), D6.3 (GK), D7.3 (GK), D8.3 (GK), D9.3 (GK)
- net CS20: now also R27.2; no longer D55.3 (GK), D56.3 (GK), D57.3 (GK), D58.3 (GK), D59.3 (GK), D60.3 (GK), D61.3 (GK), D62.3 (GK), D63.3 (GK)
- net CS21: now also R28.2; no longer D55.4 (BK), D56.4 (BK), D57.4 (BK), D58.4 (BK), D59.4 (BK), D60.4 (BK), D61.4 (BK), D62.4 (BK), D63.4 (BK)
- net CS22: now also R29.2; no longer D64.2 (RK), D65.2 (RK), D66.2 (RK), D67.2 (RK), D68.2 (RK), D69.2 (RK), D70.2 (RK), D71.2 (RK), D72.2 (RK)
- net CS23: now also R30.2; no longer D64.3 (GK), D65.3 (GK), D66.3 (GK), D67.3 (GK), D68.3 (GK), D69.3 (GK), D70.3 (GK), D71.3 (GK), D72.3 (GK)
- net CS24: now also R31.2; no longer D64.4 (BK), D65.4 (BK), D66.4 (BK), D67.4 (BK), D68.4 (BK), D69.4 (BK), D70.4 (BK), D71.4 (BK), D72.4 (BK)
- net CS25: now also R34.2; no longer D73.2 (RK), D74.2 (RK), D75.2 (RK), D76.2 (RK), D77.2 (RK), D78.2 (RK), D79.2 (RK), D80.2 (RK), D81.2 (RK)
- net CS26: now also R35.2; no longer D73.3 (GK), D74.3 (GK), D75.3 (GK), D76.3 (GK), D77.3 (GK), D78.3 (GK), D79.3 (GK), D80.3 (GK), D81.3 (GK)
- net CS27: now also R36.2; no longer D73.4 (BK), D74.4 (BK), D75.4 (BK), D76.4 (BK), D77.4 (BK), D78.4 (BK), D79.4 (BK), D80.4 (BK), D81.4 (BK)
- net CS28: now also R37.2; no longer D82.2 (RK), D83.2 (RK), D84.2 (RK), D85.2 (RK), D86.2 (RK), D87.2 (RK), D88.2 (RK), D89.2 (RK), D90.2 (RK)
- net CS29: now also R38.2; no longer D82.3 (GK), D83.3 (GK), D84.3 (GK), D85.3 (GK), D86.3 (GK), D87.3 (GK), D88.3 (GK), D89.3 (GK), D90.3 (GK)
- net CS3: now also R6.2; no longer D1.4 (BK), D2.4 (BK), D3.4 (BK), D4.4 (BK), D5.4 (BK), D6.4 (BK), D7.4 (BK), D8.4 (BK), D9.4 (BK)
- net CS30: now also R39.2; no longer D82.4 (BK), D83.4 (BK), D84.4 (BK), D85.4 (BK), D86.4 (BK), D87.4 (BK), D88.4 (BK), D89.4 (BK), D90.4 (BK)
- net CS31: no longer D91.2 (RK), D92.2 (RK), D93.2 (RK), D94.2 (RK), D95.2 (RK), D96.2 (RK), D97.2 (RK), D98.2 (RK), D99.2 (RK)
- net CS32: no longer D91.3 (GK), D92.3 (GK), D93.3 (GK), D94.3 (GK), D95.3 (GK), D96.3 (GK), D97.3 (GK), D98.3 (GK), D99.3 (GK)
- net CS33: no longer D91.4 (BK), D92.4 (BK), D93.4 (BK), D94.4 (BK), D95.4 (BK), D96.4 (BK), D97.4 (BK), D98.4 (BK), D99.4 (BK)
- net CS34: now also R43.2; no longer D100.2 (RK), D101.2 (RK), D102.2 (RK), D103.2 (RK), D104.2 (RK), D105.2 (RK), D106.2 (RK), D107.2 (RK), D108.2 (RK)
- net CS35: now also R44.2; no longer D100.3 (GK), D101.3 (GK), D102.3 (GK), D103.3 (GK), D104.3 (GK), D105.3 (GK), D106.3 (GK), D107.3 (GK)
- net CS36: now also R45.2; no longer D100.4 (BK), D101.4 (BK), D102.4 (BK), D103.4 (BK), D104.4 (BK), D105.4 (BK), D106.4 (BK), D107.4 (BK), D108.4 (BK)
- net CS37: now also R46.2; no longer D109.2 (RK), D110.2 (RK), D111.2 (RK), D112.2 (RK), D113.2 (RK), D114.2 (RK), D115.2 (RK), D116.2 (RK), D117.2 (RK)
- net CS38: now also R47.2; no longer D109.3 (GK), D110.3 (GK), D111.3 (GK), D112.3 (GK), D113.3 (GK), D114.3 (GK), D115.3 (GK), D116.3 (GK), D117.3 (GK)
- net CS39: now also R48.2; no longer D109.4 (BK), D110.4 (BK), D111.4 (BK), D112.4 (BK), D113.4 (BK), D114.4 (BK), D115.4 (BK), D116.4 (BK), D117.4 (BK)
- net CS4: now also R8.2; no longer D10.2 (RK), D11.2 (RK), D12.2 (RK), D13.2 (RK), D14.2 (RK), D15.2 (RK), D16.2 (RK), D17.2 (RK), D18.2 (RK)
- net CS5: now also R10.2; no longer D10.3 (GK), D11.3 (GK), D12.3 (GK), D13.3 (GK), D14.3 (GK), D15.3 (GK), D16.3 (GK), D17.3 (GK), D18.3 (GK)
- net CS6: now also R11.2; no longer D10.4 (BK), D11.4 (BK), D12.4 (BK), D13.4 (BK), D14.4 (BK), D15.4 (BK), D16.4 (BK), D17.4 (BK), D18.4 (BK)
- net CS7: now also R12.2; no longer D19.2 (RK), D20.2 (RK), D21.2 (RK), D22.2 (RK), D23.2 (RK), D24.2 (RK), D25.2 (RK), D26.2 (RK), D27.2 (RK)
- net CS8: now also R13.2; no longer D19.3 (GK), D20.3 (GK), D21.3 (GK), D22.3 (GK), D23.3 (GK), D24.3 (GK), D25.3 (GK), D26.3 (GK), D27.3 (GK)
- net CS9: now also R14.2; no longer D19.4 (BK), D20.4 (BK), D21.4 (BK), D22.4 (BK), D23.4 (BK), D24.4 (BK), D25.4 (BK), D26.4 (BK), D27.4 (BK)
- net GND: now also C1.2, P1.2 (P2), P2.2 (P2), P2.3 (P3), P2.4 (P4)
- net INT1: now also P2.13 (P13)
- net INT2: now also P2.14 (P14)
- net INTB: now also P2.7 (P7)
- net SA0/SDo: now also P2.11 (P11)
- net SCL_ACC: now also P2.10 (P10), P3.2 (P2)
- net SCL_MTX: now also P2.6 (P6), P3.3 (P3)
- net SDA_ACC: now also P2.9 (P9), P4.2 (P2)
- net SDA_MTX: now also P2.5 (P5), P4.3 (P3)
- net SDB: now also P2.8 (P8)
- net SW2: now also D101.1 (A), D110.1 (A), D65.1 (A), D74.1 (A), D83.1 (A), D92.1 (A)
- net at D108.3 (GK): now also D100.3 (GK), D101.3 (GK), D102.3 (GK), D103.3 (GK), D104.3 (GK), D105.3 (GK), D106.3 (GK), D107.3 (GK), R44.1
- net at D1.2 (RK): now also D2.2 (RK), D3.2 (RK), D4.2 (RK), D5.2 (RK), D6.2 (RK), D7.2 (RK), D8.2 (RK), D9.2 (RK), R1.1
- new net: D82.2 (RK), D83.2 (RK), D84.2 (RK), D85.2 (RK), D86.2 (RK), D87.2 (RK), D88.2 (RK), D89.2 (RK), D90.2 (RK), R37.1
- new net: D82.3 (GK), D83.3 (GK), D84.3 (GK), D85.3 (GK), D86.3 (GK), D87.3 (GK), D88.3 (GK), D89.3 (GK), D90.3 (GK), R38.1
- new net: D82.4 (BK), D83.4 (BK), D84.4 (BK), D85.4 (BK), D86.4 (BK), D87.4 (BK), D88.4 (BK), D89.4 (BK), D90.4 (BK), R39.1
- new net: D91.2 (RK), D92.2 (RK), D93.2 (RK), D94.2 (RK), D95.2 (RK), D96.2 (RK), D97.2 (RK), D98.2 (RK), D99.2 (RK), R40.1
- new net: D91.3 (GK), D92.3 (GK), D93.3 (GK), D94.3 (GK), D95.3 (GK), D96.3 (GK), D97.3 (GK), D98.3 (GK), D99.3 (GK), R41.1
- new net: D91.4 (BK), D92.4 (BK), D93.4 (BK), D94.4 (BK), D95.4 (BK), D96.4 (BK), D97.4 (BK), D98.4 (BK), D99.4 (BK), R42.1
- new net: D100.2 (RK), D101.2 (RK), D102.2 (RK), D103.2 (RK), D104.2 (RK), D105.2 (RK), D106.2 (RK), D107.2 (RK), D108.2 (RK), R43.1
- new net: D100.4 (BK), D101.4 (BK), D102.4 (BK), D103.4 (BK), D104.4 (BK), D105.4 (BK), D106.4 (BK), D107.4 (BK), D108.4 (BK), R45.1
- new net: D109.2 (RK), D110.2 (RK), D111.2 (RK), D112.2 (RK), D113.2 (RK), D114.2 (RK), D115.2 (RK), D116.2 (RK), D117.2 (RK), R46.1
- new net: D109.3 (GK), D110.3 (GK), D111.3 (GK), D112.3 (GK), D113.3 (GK), D114.3 (GK), D115.3 (GK), D116.3 (GK), D117.3 (GK), R47.1
- new net: D109.4 (BK), D110.4 (BK), D111.4 (BK), D112.4 (BK), D113.4 (BK), D114.4 (BK), D115.4 (BK), D116.4 (BK), D117.4 (BK), R48.1
- new net: D73.2 (RK), D74.2 (RK), D75.2 (RK), D76.2 (RK), D77.2 (RK), D78.2 (RK), D79.2 (RK), D80.2 (RK), D81.2 (RK), R34.1
- new net: D73.3 (GK), D74.3 (GK), D75.3 (GK), D76.3 (GK), D77.3 (GK), D78.3 (GK), D79.3 (GK), D80.3 (GK), D81.3 (GK), R35.1
- new net: D73.4 (BK), D74.4 (BK), D75.4 (BK), D76.4 (BK), D77.4 (BK), D78.4 (BK), D79.4 (BK), D80.4 (BK), D81.4 (BK), R36.1
- new net: D37.2 (RK), D38.2 (RK), D39.2 (RK), D40.2 (RK), D41.2 (RK), D42.2 (RK), D43.2 (RK), D44.2 (RK), D45.2 (RK), R18.1
- new net: D37.3 (GK), D38.3 (GK), D39.3 (GK), D40.3 (GK), D41.3 (GK), D42.3 (GK), D43.3 (GK), D44.3 (GK), D45.3 (GK), R19.1
- new net: D37.4 (BK), D38.4 (BK), D39.4 (BK), D40.4 (BK), D41.4 (BK), D42.4 (BK), D43.4 (BK), D44.4 (BK), D45.4 (BK), R20.1
- new net: D46.2 (RK), D47.2 (RK), D48.2 (RK), D49.2 (RK), D50.2 (RK), D51.2 (RK), D52.2 (RK), D53.2 (RK), D54.2 (RK), R21.1
- new net: D46.3 (GK), D47.3 (GK), D48.3 (GK), D49.3 (GK), D50.3 (GK), D51.3 (GK), D52.3 (GK), D53.3 (GK), D54.3 (GK), R22.1
- new net: D46.4 (BK), D47.4 (BK), D48.4 (BK), D49.4 (BK), D50.4 (BK), D51.4 (BK), D52.4 (BK), D53.4 (BK), D54.4 (BK), R23.1
- new net: D55.2 (RK), D56.2 (RK), D57.2 (RK), D58.2 (RK), D59.2 (RK), D60.2 (RK), D61.2 (RK), D62.2 (RK), D63.2 (RK), R26.1
- new net: D55.3 (GK), D56.3 (GK), D57.3 (GK), D58.3 (GK), D59.3 (GK), D60.3 (GK), D61.3 (GK), D62.3 (GK), D63.3 (GK), R27.1
- new net: D55.4 (BK), D56.4 (BK), D57.4 (BK), D58.4 (BK), D59.4 (BK), D60.4 (BK), D61.4 (BK), D62.4 (BK), D63.4 (BK), R28.1
- new net: D64.2 (RK), D65.2 (RK), D66.2 (RK), D67.2 (RK), D68.2 (RK), D69.2 (RK), D70.2 (RK), D71.2 (RK), D72.2 (RK), R29.1
- new net: D64.3 (GK), D65.3 (GK), D66.3 (GK), D67.3 (GK), D68.3 (GK), D69.3 (GK), D70.3 (GK), D71.3 (GK), D72.3 (GK), R30.1
- new net: D64.4 (BK), D65.4 (BK), D66.4 (BK), D67.4 (BK), D68.4 (BK), D69.4 (BK), D70.4 (BK), D71.4 (BK), D72.4 (BK), R31.1
- new net: D28.2 (RK), D29.2 (RK), D30.2 (RK), D31.2 (RK), D32.2 (RK), D33.2 (RK), D34.2 (RK), D35.2 (RK), D36.2 (RK), R15.1
- new net: D28.3 (GK), D29.3 (GK), D30.3 (GK), D31.3 (GK), D32.3 (GK), D33.3 (GK), D34.3 (GK), D35.3 (GK), D36.3 (GK), R16.1
- new net: D28.4 (BK), D29.4 (BK), D30.4 (BK), D31.4 (BK), D32.4 (BK), D33.4 (BK), D34.4 (BK), D35.4 (BK), D36.4 (BK), R17.1
- new net: D10.2 (RK), D11.2 (RK), D12.2 (RK), D13.2 (RK), D14.2 (RK), D15.2 (RK), D16.2 (RK), D17.2 (RK), D18.2 (RK), R8.1
- new net: D10.3 (GK), D11.3 (GK), D12.3 (GK), D13.3 (GK), D14.3 (GK), D15.3 (GK), D16.3 (GK), D17.3 (GK), D18.3 (GK), R10.1
- new net: D10.4 (BK), D11.4 (BK), D12.4 (BK), D13.4 (BK), D14.4 (BK), D15.4 (BK), D16.4 (BK), D17.4 (BK), D18.4 (BK), R11.1
- new net: D19.2 (RK), D20.2 (RK), D21.2 (RK), D22.2 (RK), D23.2 (RK), D24.2 (RK), D25.2 (RK), D26.2 (RK), D27.2 (RK), R12.1
- new net: D19.3 (GK), D20.3 (GK), D21.3 (GK), D22.3 (GK), D23.3 (GK), D24.3 (GK), D25.3 (GK), D26.3 (GK), D27.3 (GK), R13.1
- new net: D19.4 (BK), D20.4 (BK), D21.4 (BK), D22.4 (BK), D23.4 (BK), D24.4 (BK), D25.4 (BK), D26.4 (BK), D27.4 (BK), R14.1
- new net: D1.3 (GK), D2.3 (GK), D3.3 (GK), D4.3 (GK), D5.3 (GK), D6.3 (GK), D7.3 (GK), D8.3 (GK), D9.3 (GK), R5.1
- new net: D1.4 (BK), D2.4 (BK), D3.4 (BK), D4.4 (BK), D5.4 (BK), D6.4 (BK), D7.4 (BK), D8.4 (BK), D9.4 (BK), R6.1
- new net GPIO1: P1.5 (P5), P2.17 (P17)
- new net GPIO2: P1.6 (P6), P2.18 (P18)
- new net SCL_SAO: P1.4 (P4), P2.16 (P16), P3.1 (P1), R25.2
- new net SDA_SAO: P1.3 (P3), P2.15 (P15), P4.1 (P1), R24.2
Other:
- note added: "Accelerometer"
- note added: "Connectors"
- note added: "LED Matrix Driver"
- note added: "Shitty Addon Module"
- moved on the sheet: C4, R32, R33, U2

Commit message: more routing on prototype
Connections:
- net CS31: now also R40.2
- net CS32: now also R41.2
- net CS33: now also R42.2
Changed lines of the file:
@@
 Wire Wire Line
 	7950 12600 7950 12650
+Wire Wire Line
+	1750 11550 1900 11550
+Wire Wire Line
+	1750 11750 1900 11750
+Wire Wire Line
+	1750 11950 1900 11950
 $EndSCHEMATC
