File: board/lixie/lixie.sch (KiCad schematic (older format))
At the start: 44 parts, among them P1 USB_OTG, P2 CONN_01X04, SW1 SW_Push, U1 IS31FL3738, U2 MAX40200, U3 MIC550x, U4 STM32L073xZ

Commit message: made artwork, rewired the LEDs
Parts:
- F1, F2, F3: footprint Fuse:Fuse_0805_2012Metric_Pad1.15x1.40mm_HandSolder -> Fuse:Fuse_1206_3216Metric_Pad1.42x1.75mm_HandSolder
Changed lines of the file:
@@
 F 0 "F2" V 11950 11050 50  0000 C CNN
 F 1 "Polyfuse" V 12150 11050 50  0000 C CNN
-F 2 "Fuse:Fuse_0805_2012Metric_Pad1.15x1.40mm_HandSolder" H 12100 10850 50  0001 L CNN
+F 2 "Fuse:Fuse_1206_3216Metric_Pad1.42x1.75mm_HandSolder" H 12100 10850 50  0001 L CNN
 F 3 "" H 12050 11050 50  0001 C CNN
 	1    12050 11050
@@
 F 0 "F3" V 10000 12200 50  0000 C CNN
 F 1 "Polyfuse" V 10200 12200 50  0000 C CNN
-F 2 "Fuse:Fuse_0805_2012Metric_Pad1.15x1.40mm_HandSolder" H 10150 12000 50  0001 L CNN
+F 2 "Fuse:Fuse_1206_3216Metric_Pad1.42x1.75mm_HandSolder" H 10150 12000 50  0001 L CNN
 F 3 "" H 10100 12200 50  0001 C CNN
 	1    10100 12200
@@
 F 0 "F1" V 10000 10800 50  0000 C CNN
 F 1 "Polyfuse" V 10200 10800 50  0000 C CNN
-F 2 "Fuse:Fuse_0805_2012Metric_Pad1.15x1.40mm_HandSolder" H 10150 10600 50  0001 L CNN
+F 2 "Fuse:Fuse_1206_3216Metric_Pad1.42x1.75mm_HandSolder" H 10150 10600 50  0001 L CNN
 F 3 "" H 10100 10800 50  0001 C CNN
 	1    10100 10800
