File: board/prototype/frkbmb28.sch (KiCad schematic (older format))
At the start: 175 parts, among them P1 SHITTY_ADD_ON, P2 MCU_CONNECTOR, P3 SCL_JMP, P4 SDA_JMP, U1 IS31FL3741, U2 LIS2HH12

Commit message: made matrix for new LED driver. TODO: Redo the accelerometer footprint because it's slightly off due to how the wizard works
Parts:
- removed C1: 10uF, SMD_Packages:SMD-1210_Pol, symbol CP
- removed D1, D10, D100, D101, D102, D103, D104, D105, D106, D107, D108, D109, D11, D110, D111, D112, D113, D114, D115, D116, D117, D12, D13, D14, D15, D16, D17, D18, D19, D2, D20, D21, D22, D23, D24, D25, D26, D27, D28, D29, D3, D30, D31, D32, D33, D34, D35, D36, D37, D38, D39, D4, D40, D41, D42, D43, D44, D45, D46, D47, D48, D49, D5, D50, D51, D52, D53, D54, D55, D56, D57, D58, D59, D6, D60, D61, D62, D63, D64, D65, D66, D67, D68, D69, D7, D70, D71, D72, D73, D74, D75, D76, D77, D78, D79, D8, D80, D81, D82, D83, D84, D85, D86, D87, D88, D89, D9, D90, D91, D92, D93, D94, D95, D96, D97, D98, D99: LED_ARGB, frkbmb:0606_RGB_COMM_ANODE, symbol LED_ARGB
- removed P2: MCU_CONNECTOR, Pin_Headers:Pin_Header_Straight_1x18, symbol CONN_01X18
- removed R1, R10, R11, R12, R13, R14, R15, R16, R17, R18, R19, R20, R21, R22, R23, R26, R27, R28, R29, R30, R31, R34, R35, R36, R37, R38, R39, R40, R41, R42, R43, R44, R45, R46, R47, R48, R5, R6, R8: R, Resistors_SMD:R_0805_HandSoldering, symbol R
- removed R4, R7: 100k, Resistors_SMD:R_0603_HandSoldering, symbol R
- removed R9: 20k, Resistors_SMD:R_0603_HandSoldering, symbol R
- removed U1: IS31FL3741, frkbmb:IS31FL3741, symbol IS31FL3741
- added C?: 100nF, Capacitors_SMD:C_0603_HandSoldering, symbol C
- added C?: 220nF, Capacitors_SMD:C_0603_HandSoldering, symbol C
- added D? (x144): LED, symbol LED
- added P?: MCU_CONNECTOR, symbol CONN_01X20
- added R?: 4.7k, Resistors_SMD:R_0603_HandSoldering, symbol R
- added R? (x2): 100k, Resistors_SMD:R_0603_HandSoldering, symbol R
- added U?: IS31FL3731, symbol IS31FL3731
- R2, R3: value 1k -> 4.7k
Connections:
- net labels added: AUD, CA1, CA2, CA3, CA4, CA5, CA6, CA7, CA8, CA9, CB1, CB2, CB3, CB4, CB5, CB6, CB7, CB8, CB9
- net labels removed: CS1, CS10, CS11, CS12, CS13, CS14, CS15, CS16, CS17, CS18, CS19, CS2, CS20, CS21, CS22, CS23, CS24, CS25, CS26, CS27, CS28, CS29, CS3, CS30, CS31, CS32, CS33, CS34, CS35, CS36, CS37, CS38, CS39, CS4, CS5, CS6, CS7, CS8, CS9, SW1, SW2, SW3, SW4, SW5, SW6, SW7, SW8, SW9
- wire segments 353 -> 279
Other:
- note removed: "LED Matrix Driver"
- moved on the sheet: C2, C3, C4, P1, P3, P4, R2, R24, R25, R3, R32, R33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

Commit message: ready to start laying out new board
Parts:
- D1, D10, D100, D101, D102, D103, D104, D105, D106, D107, D108, D109, D11, D110, D111, D112, D113, D114, D115, D116, D117, D118, D119, D12, D120, D121, D122, D123, D124, D125, D126, D127, D128, D129, D13, D130, D131, D132, D133, D134, D135, D136, D137, D138, D139, D14, D140, D141, D142, D143, D144, D15, D16, D17, D18, D19, D2, D20, D21, D22, D23, D24, D25, D26, D27, D28, D29, D3, D30, D31, D32, D33, D34, D35, D36, D37, D38, D39, D4, D40, D41, D42, D43, D44, D45, D46, D47, D48, D49, D5, D50, D51, D52, D53, D54, D55, D56, D57, D58, D59, D6, D60, D61, D62, D63, D64, D65, D66, D67, D68, D69, D7, D70, D71, D72, D73, D74, D75, D76, D77, D78, D79, D8, D80, D81, D82, D83, D84, D85, D86, D87, D88, D89, D9, D90, D91, D92, D93, D94, D95, D96, D97, D98, D99: renamed from D?; footprint (none) -> LEDs:LED_0805
- P2: renamed from P?; footprint (none) -> Pin_Headers:Pin_Header_Straight_1x20
- U1: renamed from U?; footprint (none) -> frkbmb:IS31FL3731C
- U2: footprint frkbmb:LIS2HH12 -> frkbmb:LIS2HH12-NEW
- gave numbers to parts that had none: 5

Commit message: ready to export gerbers, waiting on approval from group
Connections:
- net SAO/SDO is gone; now on net SA0_SDO: R32.2, U2.3 (SA0/SDO)
- net CB1: now also U1.7 (CB1)
- net CB2: now also U1.8 (CB2)
- net CB3: now also U1.9 (CB3)
- net CB4: now also U1.10 (CB4)
- net CB5: now also U1.11 (CB5)
- net CB6: now also U1.12 (CB6)
- net CB7: now also U1.13 (CB7)
- net CB8: now also U1.14 (CB8)
- net CB9: now also U1.15 (CB9)
- net SDB: now also R4.2
- net SA0/SDo renamed SA0_SDO
Changed lines of the file:
@@
 $EndComp
 Text Label 1950 8550 2    60   ~ 0
-SAO/SDO
+SA0_SDO
 Text Label 1950 8650 2    60   ~ 0
 CS
@@
 SCL_ACC
 Text Label 3100 11650 2    60   ~ 0
-SA0/SDo
+SA0_SDO
 Text Label 3100 11750 2    60   ~ 0
 CS
@@
 Text Label 3100 11350 2    60   ~ 0
 AUD
+Wire Wire Line
+	3950 1800 4150 1800
+Wire Wire Line
+	3950 1900 4150 1900
+Wire Wire Line
+	3950 2000 4150 2000
+Wire Wire Line
+	3950 2100 4150 2100
+Wire Wire Line
+	3950 2200 4150 2200
+Wire Wire Line
+	3950 2300 4150 2300
+Wire Wire Line
+	3950 2400 4150 2400
+Wire Wire Line
+	3950 2500 4150 2500
+Wire Wire Line
+	3950 2600 4150 2600
+Connection ~ 4150 1800
+Connection ~ 4150 1900
+Connection ~ 4150 2000
+Connection ~ 4150 2100
+Connection ~ 4150 2200
+Connection ~ 4150 2300
+Connection ~ 4150 2400
+Connection ~ 4150 2500
+Connection ~ 4150 2600
+Text Label 4150 1800 0    60   ~ 0
+CB9
+Text Label 4150 1900 0    60   ~ 0
+CB8
+Text Label 4150 2000 0    60   ~ 0
+CB7
+Text Label 4150 2100 0    60   ~ 0
+CB6
+Text Label 4150 2200 0    60   ~ 0
+CB5
+Text Label 4150 2300 0    60   ~ 0
+CB4
+Text Label 4150 2400 0    60   ~ 0
+CB3
+Text Label 4150 2500 0    60   ~ 0
+CB2
+Text Label 4150 2600 0    60   ~ 0
+CB1
+Connection ~ 1200 1750
 $EndSCHEMATC

Commit message: working on a cancelled badge
Parts:
- C1, C2, C3, C4, C5: symbol C -> frkbmb28-rescue:C
- D1, D10, D100, D101, D102, D103, D104, D105, D106, D107, D108, D109, D11, D110, D111, D112, D113, D114, D115, D116, D117, D118, D119, D12, D120, D121, D122, D123, D124, D125, D126, D127, D128, D129, D13, D130, D131, D132, D133, D134, D135, D136, D137, D138, D139, D14, D140, D141, D142, D143, D144, D15, D16, D17, D18, D19, D2, D20, D21, D22, D23, D24, D25, D26, D27, D28, D29, D3, D30, D31, D32, D33, D34, D35, D36, D37, D38, D39, D4, D40, D41, D42, D43, D44, D45, D46, D47, D48, D49, D5, D50, D51, D52, D53, D54, D55, D56, D57, D58, D59, D6, D60, D61, D62, D63, D64, D65, D66, D67, D68, D69, D7, D70, D71, D72, D73, D74, D75, D76, D77, D78, D79, D8, D80, D81, D82, D83, D84, D85, D86, D87, D88, D89, D9, D90, D91, D92, D93, D94, D95, D96, D97, D98, D99: symbol LED -> frkbmb28-rescue:LED
- P1: symbol CONN_02X03 -> frkbmb28-rescue:CONN_02X03
- P2: symbol CONN_01X20 -> frkbmb28-rescue:CONN_01X20
- P3, P4: symbol CONN_01X03 -> frkbmb28-rescue:CONN_01X03
- R1, R2, R24, R25, R3, R32, R33, R4, R5: symbol R -> frkbmb28-rescue:R
- U1: symbol IS31FL3731 -> frkbmb28:IS31FL3731
- U2: symbol LIS2HH12 -> frkbmb28:LIS2HH12
Connections:
- net CA7: no longer D54.2 (A)
- net CB7: no longer D62.2 (A)
